File: HAS-CT-Board.sch (KiCad schematic (older format))
At the start: 63 parts, among them J1 HAS-CT1, J2 HAS-CT2, J3 HAS-CT3, J4 SMB, J5 SMB, J6 SMB, P1 Conn_WallPlug, U1 NJM4580, U2 NJM4580, U3 NJM4580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

Commit message: Add: 配線のみ完了
Parts:
- added H1, H2, H3, H4: MountingHole, myLib:MountingHole_3.2mm_M3_noResist, symbol Mechanical:MountingHole
Changed lines of the file:
@@
 	-1   0    0    1
 $EndComp
+$Comp
+L Mechanical:MountingHole H1
+U 1 1 61502E2E
+P 2000 2000
+F 0 "H1" H 2100 2046 50  0000 L CNN
+F 1 "MountingHole" H 2100 1955 50  0000 L CNN
+F 2 "myLib:MountingHole_3.2mm_M3_noResist" H 2000 2000 50  0001 C CNN
+F 3 "~" H 2000 2000 50  0001 C CNN
+	1    2000 2000
+	1    0    0    -1
+$EndComp
+$Comp
+L Mechanical:MountingHole H3
+U 1 1 6150486E
+P 3000 2000
+F 0 "H3" H 3100 2046 50  0000 L CNN
+F 1 "MountingHole" H 3100 1955 50  0000 L CNN
+F 2 "myLib:MountingHole_3.2mm_M3_noResist" H 3000 2000 50  0001 C CNN
+F 3 "~" H 3000 2000 50  0001 C CNN
+	1    3000 2000
+	1    0    0    -1
+$EndComp
+$Comp
+L Mechanical:MountingHole H2
+U 1 1 61504D8B
+P 2000 2500
+F 0 "H2" H 2100 2546 50  0000 L CNN
+F 1 "MountingHole" H 2100 2455 50  0000 L CNN
+F 2 "myLib:MountingHole_3.2mm_M3_noResist" H 2000 2500 50  0001 C CNN
+F 3 "~" H 2000 2500 50  0001 C CNN
+	1    2000 2500
+	1    0    0    -1
+$EndComp
+$Comp
+L Mechanical:MountingHole H4
+U 1 1 61505176
+P 3000 2500
+F 0 "H4" H 3100 2546 50  0000 L CNN
+F 1 "MountingHole" H 3100 2455 50  0000 L CNN
+F 2 "myLib:MountingHole_3.2mm_M3_noResist" H 3000 2500 50  0001 C CNN
+F 3 "~" H 3000 2500 50  0001 C CNN
+	1    3000 2500
+	1    0    0    -1
+$EndComp
 $EndSCHEMATC
