File: HAS-CT-Board.kicad_pcb (KiCad board)
At the start: 2 copper layers, 100 x 100 mm, 67 parts, among them J1 HAS-CT1, J2 HAS-CT2, J3 HAS-CT3, J4 SMB, J5 SMB, J6 SMB, P1 Conn_WallPlug, U1 NJM4580, U2 NJM4580, U3 NJM4580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

Commit message: Update: PCB
Routing:
- net +15V: track 331.1 -> 332.7 mm
- net GND: track 409.5 -> 408.8 mm
Other:
- board text added: "GND"
